Commit message: fix poltmetis dependcies

File: role_ros2/robot_ik/franka/fr3.urdf (robot description, URDF)
Before this commit: robot fr3_robot, 10 links, 7 joints
Links:
- removed link fr3_panda_link8
- added link base_link, mass 0.001
- link fr3_panda_hand: geometry collision mesh filename=package://role_ros2/robot_ik/franka/mesh/hand.obj; visual mesh filename=package://role_ros2/robot_ik/franka/mesh/hand.obj
- link fr3_panda_link0: geometry collision mesh filename=package://role_ros2/robot_ik/franka/mesh/link0.obj; visual mesh filename=package://role_ros2/robot_ik/franka/mesh/link0.obj
- link fr3_panda_link1: geometry collision mesh filename=package://role_ros2/robot_ik/franka/mesh/link1.obj; visual mesh filename=package://role_ros2/robot_ik/franka/mesh/link1.obj
- link fr3_panda_link2: geometry collision mesh filename=package://role_ros2/robot_ik/franka/mesh/link2.obj; visual mesh filename=package://role_ros2/robot_ik/franka/mesh/link2.obj
- link fr3_panda_link3: geometry collision mesh filename=package://role_ros2/robot_ik/franka/mesh/link3.obj; visual mesh filename=package://role_ros2/robot_ik/franka/mesh/link3.obj
- link fr3_panda_link4: geometry collision mesh filename=package://role_ros2/robot_ik/franka/mesh/link4.obj; visual mesh filename=package://role_ros2/robot_ik/franka/mesh/link4.obj
- link fr3_panda_link5: geometry collision mesh filename=package://role_ros2/robot_ik/franka/mesh/link5.obj; visual mesh filename=package://role_ros2/robot_ik/franka/mesh/link5.obj
- link fr3_panda_link6: geometry collision mesh filename=package://role_ros2/robot_ik/franka/mesh/link6.obj; visual mesh filename=package://role_ros2/robot_ik/franka/mesh/link6.obj
- link fr3_panda_link7: geometry collision mesh filename=package://role_ros2/robot_ik/franka/mesh/link7.obj; visual mesh filename=package://role_ros2/robot_ik/franka/mesh/link7.obj
Joints:
- added joint fr3_base_joint: type fixed, parent base_link, child fr3_panda_link0, origin xyz=0.0 0.0 0.0 rpy=0 0 0
- added joint fr3_panda_hand_fixed_joint: type fixed, parent fr3_panda_link7, child fr3_panda_hand, origin xyz=0.0 0.0 0.107 rpy=0.0 0.0 -0.785398163397

Commit message: add vr node and teleoperation node

File: role_ros2/robot_ik/franka/fr3.urdf (robot description, URDF)
Before this commit: robot fr3_robot, 10 links, 9 joints
Links:
- added link fr3_panda_link8, mass 0.0
Joints:
- removed joint fr3_panda_hand_fixed_joint
- added joint fr3_panda_hand_joint: type fixed, parent fr3_panda_link8, child fr3_panda_hand, origin xyz=0 0 0 rpy=0 0 -0.785398163397
- added joint fr3_panda_joint8: type fixed, parent fr3_panda_link7, child fr3_panda_link8, origin xyz=0 0 0.107 rpy=0 0 0, axis 0 0 0
